File: airdata.kicad_sch (KiCad schematic)
At the start: 7 parts, among them J1 AE-MICRO-SD-DIP, U1 DPS310, U2 SeeeduinoXIAO

Commit message: Revert "update to 24th add R"
Parts:
- removed JP1: SolderJumper_2_Open, symbol Jumper:SolderJumper_2_Open
- removed R1: 1k, symbol Device:R
Connections:
- no-connect marks 9 -> 0
Other:
- company: TORICA-24th -> (none)
- title: AirData -> (none)
